File: RS1_PCB_main.kicad_pcb (KiCad board)
At the start: 2 copper layers, 47.5 x 39.5 mm, 51 parts, among them J1 Conn_01x05, J3 Connector, USB-TYPE-C-16P, J5 Conn_01x02, J7 Conn_01x02, J8 Conn_01x02, Q4 2N7002, SW3 GT-TC172A-H035-L1 (PWR BTN), U1 ESP32-C6-WROOM-1, U17 ME6217C33M5G, U2 USBLC6-2SC6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

Commit message: small adj
Parts:
- moved Q4 1.82 mm to (188.1, 51.5)
- moved C15 0.88 mm to (186.2, 50.8), turned to 180 degrees
Routing:
- net Net-(Q4-D): track 3.88 -> 4.77 mm
Changed lines of the file:
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@@
 	(footprint "PCM_JLCPCB:Q_SOT-23"
 		(layer "F.Cu")
-		(at 189.52 50.36)
+		(at 188.14 51.55)
 		(descr "SOT, 3 Pin (https://www.jedec.org/system/files/docs/to-236h.pdf variant AB), generated with kicad-footprint-generator ipc_gullwing_generator.py")
 		(tags "SOT TO_SOT_SMD")
@@
 	(footprint "PCM_JLCPCB:C_0603"
 		(layer "B.Cu")
-		(at 186.92 50.3 90)
+		(at 186.2 50.8 180)
 		(descr "Capacitor SMD 0603 (1608 Metric), square (rectangular) end terminal, IPC_7351 nominal, (Body size source: IPC-SM-782 page 76, https://www.pcb-3d.com/wordpress/wp-content/uploads/ipc-sm-782a_amendment_1_and_2.pdf), generated with kicad-footprint-generator")
 		(tags "capacitor")
 		(property "Reference" "C15"
-			(at 2.16 1.55 180)
+			(at 2.16 1.55 90)
 			(layer "B.SilkS")
 			(effects
@@
 		)
 		(property "Value" "100nF"
-			(at 0 -1.43 90)
+			(at 0 -1.43 0)
 			(layer "B.Fab")
 			(effects
@@
 		)
 		(property "Datasheet" "https://www.lcsc.com/datasheet/lcsc_datasheet_2211101700_YAGEO-CC0603KRX7R9BB104_C14663.pdf"
-			(at 0 0 270)
+			(at 0 0 0)
 			(unlocked yes)
 			(layer "B.Fab")
@@
 		)
 		(property "Description" "50V 100nF X7R ±10% 0603 Multilayer Ceramic Capacitors MLCC - SMD/SMT ROHS"
-			(at 0 0 270)
+			(at 0 0 0)
 			(unlocked yes)
 			(layer "B.Fab")
@@
 		)
 		(property "LCSC" "C14663"
-			(at 0 0 270)
+			(at 0 0 0)
 			(unlocked yes)
 			(layer "B.Fab")
@@
 		)
 		(property "Stock" "70324515"
-			(at 0 0 270)
+			(at 0 0 0)
 			(unlocked yes)
 			(layer "B.Fab")
@@
 		)
 		(property "Price" "0.006USD"
-			(at 0 0 270)
+			(at 0 0 0)
 			(unlocked yes)
 			(layer "B.Fab")
@@
 		)
 		(property "Process" "SMT"
-			(at 0 0 270)
+			(at 0 0 0)
 			(unlocked yes)
 			(layer "B.Fab")
@@
 		)
 		(property "Minimum Qty" "20"
-			(at 0 0 270)
+			(at 0 0 0)
 			(unlocked yes)
 			(layer "B.Fab")
@@
 		)
 		(property "Attrition Qty" "10"
-			(at 0 0 270)
+			(at 0 0 0)
 			(unlocked yes)
 			(layer "B.Fab")
@@
 		)
 		(property "Class" "Basic Component"
-			(at 0 0 270)
+			(at 0 0 0)
 			(unlocked yes)
 			(layer "B.Fab")
@@
 		)
 		(property "Category" "Capacitors,Multilayer Ceramic Capacitors MLCC - SMD/SMT"
-			(at 0 0 270)
+			(at 0 0 0)
 			(unlocked yes)
 			(layer "B.Fab")
@@
 		)
 		(property "Manufacturer" "YAGEO"
-			(at 0 0 270)
+			(at 0 0 0)
 			(unlocked yes)
 			(layer "B.Fab")
@@
 		)
 		(property "Part" "CC0603KRX7R9BB104"
-			(at 0 0 270)
+			(at 0 0 0)
 			(unlocked yes)
 			(layer "B.Fab")
@@
 		)
 		(property "Voltage Rated" "50V"
-			(at 0 0 270)
+			(at 0 0 0)
 			(unlocked yes)
 			(layer "B.Fab")
@@
 		)
 		(property "Tolerance" "±10%"
-			(at 0 0 270)
+			(at 0 0 0)
 			(unlocked yes)
 			(layer "B.Fab")
@@
 		)
 		(property "Capacitance" "100nF"
-			(at 0 0 270)
+			(at 0 0 0)
 			(unlocked yes)
 			(layer "B.Fab")
@@
 		)
 		(property "Temperature Coefficient" "X7R"
-			(at 0 0 270)
+			(at 0 0 0)
 			(unlocked yes)
 			(layer "B.Fab")
@@
 		(attr smd)
 		(fp_line
-			(start 1.4 -0.6)
-			(end -1.4 -0.6)
+			(start 1.4 0.6)
+			(end 1.4 -0.6)
 			(stroke
 				(width 0.05)
@@
 		)
 		(fp_line
-			(start -1.4 -0.6)
-			(end -1.4 0.6)
+			(start 1.4 -0.6)
+			(end -1.4 -0.6)
 			(stroke
 				(width 0.05)
@@
 		)
 		(fp_line
-			(start 1.4 0.6)
-			(end 1.4 -0.6)
+			(start -1.4 0.6)
+			(end 1.4 0.6)
 			(stroke
 				(width 0.05)
@@
 		)
 		(fp_line
-			(start -1.4 0.6)
-			(end 1.4 0.6)
+			(start -1.4 -0.6)
+			(end -1.4 0.6)
 			(stroke
 				(width 0.05)
@@
 		)
 		(fp_line
-			(start 0.8 -0.4)
-			(end -0.8 -0.4)
+			(start 0.8 0.4)
+			(end 0.8 -0.4)
 			(stroke
 				(width 0.1)
@@
 		)
 		(fp_line
-			(start -0.8 -0.4)
-			(end -0.8 0.4)
+			(start 0.8 -0.4)
+			(end -0.8 -0.4)
 			(stroke
 				(width 0.1)
@@
 		)
 		(fp_line
-			(start 0.8 0.4)
-			(end 0.8 -0.4)
+			(start -0.8 0.4)
+			(end 0.8 0.4)
 			(stroke
 				(width 0.1)
@@
 		)
 		(fp_line
-			(start -0.8 0.4)
-			(end 0.8 0.4)
+			(start -0.8 -0.4)
+			(end -0.8 0.4)
 			(stroke
 				(width 0.1)
@@
 		)
 		(fp_text user "${REFERENCE}"
-			(at 0 0 90)
+			(at 0 0 0)
 			(layer "B.Fab")
 			(effects
@@
 		)
 		(pad "1" smd roundrect
-			(at -0.78 0 90)
+			(at -0.78 0 180)
 			(size 0.9 0.95)
 			(layers "B.Cu" "B.Mask" "B.Paste")
@@
 		)
 		(pad "2" smd roundrect
-			(at 0.78 0 90)
+			(at 0.78 0 180)
 			(size 0.9 0.95)
 			(layers "B.Cu" "B.Mask" "B.Paste")
@@
 	)
 	(via
-		(at 184.9 49.8)
+		(at 184.8 49.3)
 		(size 0.6)
 		(drill 0.3)
@@
 	)
 	(segment
-		(start 192.32 51.8)
-		(end 192.32 52.41)
+		(start 192.32 52.41)
+		(end 191.9 52.83)
 		(width 0.2)
 		(layer "F.Cu")
@@
 	)
 	(segment
-		(start 190.46 50.36)
-		(end 190.46 50.74)
+		(start 191.28 51.56)
+		(end 191.5 51.56)
 		(width 0.2)
 		(layer "F.Cu")
@@
 	)
 	(segment
-		(start 190.46 50.74)
-		(end 191.28 51.56)
+		(start 192.08 51.56)
+		(end 192.32 51.8)
 		(width 0.2)
 		(layer "F.Cu")
@@
 	)
 	(segment
-		(start 191.28 51.56)
-		(end 192.08 51.56)
+		(start 191.5 51.56)
+		(end 191.49 51.55)
 		(width 0.2)
 		(layer "F.Cu")
@@
 	)
 	(segment
-		(start 192.32 52.41)
-		(end 191.9 52.83)
+		(start 191.5 51.56)
+		(end 192.08 51.56)
 		(width 0.2)
 		(layer "F.Cu")
@@
 	)
 	(segment
-		(start 192.08 51.56)
-		(end 192.32 51.8)
+		(start 191.49 51.55)
+		(end 189.08 51.55)
 		(width 0.2)
 		(layer "F.Cu")
@@
 	)
 	(segment
-		(start 180.45 61.55)
-		(end 179.7 62.3)
+		(start 192.32 51.8)
+		(end 192.32 52.41)
 		(width 0.2)
 		(layer "F.Cu")
-		(net 32)
+		(net 31)
 	)
 	(segment
-		(start 187.19 49.41)
-		(end 185.95 50.65)
+		(start 187.2 50.6)
+		(end 188.1 49.7)
 		(width 0.2)
 		(layer "F.Cu")
@@
 	)
 	(segment
-		(start 185.95 52.6)
-		(end 180.45 58.1)
+		(start 180.45 57.05)
+		(end 180.45 61.55)
 		(width 0.2)
 		(layer "F.Cu")
@@
 	)
 	(segment
-		(start 191.89 49.41)
-		(end 188.58 49.41)
+		(start 180.45 61.55)
+		(end 179.7 62.3)
 		(width 0.2)
 		(layer "F.Cu")
@@
 	)
 	(segment
-		(start 185.95 50.65)
-		(end 185.95 52.6)
+		(start 193.2 49.7)
+		(end 192.2 49.7)
 		(width 0.2)
 		(layer "F.Cu")
@@
 	)
 	(segment
-		(start 180.45 58.1)
-		(end 180.45 61.55)
+		(start 184.9 52.6)
+		(end 184.9 51.6)
 		(width 0.2)
 		(layer "F.Cu")
@@
 	)
 	(segment
-		(start 193.2 49.7)
-		(end 192.2 49.7)
+		(start 184.9 51.6)
+		(end 185.9 50.6)
 		(width 0.2)
 		(layer "F.Cu")
@@
 	)
 	(segment
-		(start 188.58 49.41)
-		(end 187.19 49.41)
+		(start 185.9 50.6)
+		(end 187.2 50.6)
 		(width 0.2)
 		(layer "F.Cu")
@@
 	)
 	(segment
-		(start 179.7 62.3)
-		(end 179.5 62.3)
+		(start 188.1 49.7)
+		(end 192.2 49.7)
 		(width 0.2)
 		(layer "F.Cu")
@@
 	)
 	(segment
-		(start 191.9 49.4)
-		(end 191.89 49.41)
+		(start 179.7 62.3)
+		(end 179.5 62.3)
 		(width 0.2)
 		(layer "F.Cu")
@@
 	)
 	(segment
-		(start 192.2 49.7)
-		(end 191.9 49.4)
+		(start 184.9 52.6)
+		(end 180.45 57.05)
 		(width 0.2)
 		(layer "F.Cu")
@@
 		(polygon
 			(pts
-				(xy 142.15 36.6) (xy 141.65 85.8) (xy 200.6 86) (xy 200.95 36.45) (xy 142.2 36.6)
+				(xy 197.087665 37.592734) (xy 197.587665 86.792734) (xy 138.637665 86.992734) (xy 138.287665 37.442734)
+				(xy 197.037665 37.592734)
 			)
 		)
